File: pcb/tft_pam_support.kicad_pcb (KiCad board)
At the start: 2 copper layers, 36.1 x 34.9 mm, 6 parts, among them J1 JST-PH2, J2 Conn_01x08, U1 TFT_1.8_no_SD, U2 PAM8302AAD

Commit message: replaced footprint for JST-connector THT->SMD
Parts:
- J1: footprint Connector_JST:JST_PH_S2B-PH-K_1x02_P2.00mm_Horizontal -> Connector_JST:JST_PH_S2B-PH-SM4-TB_1x02-1MP_P2.00mm_Horizontal
- moved J1 4.08 mm to (106.4, 83.6)
Routing:
- net Net-(J1-Pad2): track 2.97 -> 4.14 mm
- net Net-(J1-Pad1): track 3.12 -> 4.20 mm
