File: pcb/tft_pam_support.kicad_sch (KiCad schematic)
At the start: 6 parts, among them J1 JST-PH2, J2 Conn_01x08, U1 TFT_1.8_no_SD, U2 PAM8302AAD

Commit message: replaced footprint for JST-connector THT->SMD
Parts:
- J1: footprint Connector_JST:JST_PH_S2B-PH-K_1x02_P2.00mm_Horizontal -> Connector_JST:JST_PH_S2B-PH-SM4-TB_1x02-1MP_P2.00mm_Horizontal
Changed lines of the file:
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@@
   (title_block
     (title "Support PCB for PAM8302A and TFT")
-    (date "2022-07-07")
-    (rev "1")
+    (date "2022-07-28")
+    (rev "2")
     (company "Bernhard Bablok")
     (comment 1 "https://github.com/bablokb/christmas-box")
@@
       (effects (font (size 1.27 1.27)) (justify left))
     )
-    (property "Footprint" "Connector_JST:JST_PH_S2B-PH-K_1x02_P2.00mm_Horizontal" (id 2) (at 163.83 62.865 0)
+    (property "Footprint" "Connector_JST:JST_PH_S2B-PH-SM4-TB_1x02-1MP_P2.00mm_Horizontal" (id 2) (at 163.83 62.865 0)
       (effects (font (size 1.27 1.27)) hide)
     )
@@
     )
     (path "/54f34bf7-2090-40f1-94b7-7f1bea5601b1"
-      (reference "J1") (unit 1) (value "JST-PH2") (footprint "Connector_JST:JST_PH_S2B-PH-K_1x02_P2.00mm_Horizontal")
+      (reference "J1") (unit 1) (value "JST-PH2") (footprint "Connector_JST:JST_PH_S2B-PH-SM4-TB_1x02-1MP_P2.00mm_Horizontal")
     )
     (path "/4f6efd07-434c-4726-9dfe-6ecc334d3305"
